Commit message: describe robot.urdf based on gyroboy design

File: ev3_robots/ev3_robot_gyro_car/robot.urdf (robot description, URDF)
Before this commit: robot ev3_robot_gyro_car, 111 links, 110 joints
Links:
- removed link accel_link
- removed link ref_0_link
- removed link ref_100_link
- removed link ref_101_link
- removed link ref_102_link
- removed link ref_103_link
- removed link ref_104_link
- removed link ref_105_link
- removed link ref_106_link
- removed link ref_10_link
- removed link ref_11_link
- removed link ref_11_link_hub
- removed link ref_12_link
- removed link ref_13_link
- removed link ref_14_link
- removed link ref_15_link
- removed link ref_16_link
- removed link ref_17_link
- removed link ref_18_link
- removed link ref_18_link_hub
- removed link ref_19_link
- removed link ref_1_link
- removed link ref_20_link
- removed link ref_21_link
- removed link ref_22_link
- removed link ref_23_link
- removed link ref_24_link
- removed link ref_24_link_hub
- removed link ref_25_link
- removed link ref_26_link
- removed link ref_27_link
- removed link ref_28_link
- removed link ref_29_link
- removed link ref_2_link
- removed link ref_30_link
- removed link ref_31_link
- removed link ref_32_link
- removed link ref_33_link
- removed link ref_34_link
- removed link ref_35_link
- removed link ref_36_link
- removed link ref_37_link
- removed link ref_38_link
- removed link ref_39_link
- removed link ref_40_link
- removed link ref_41_link
- removed link ref_42_link
- removed link ref_43_link
- removed link ref_44_link
- removed link ref_45_link
- removed link ref_46_link
- removed link ref_47_link
- removed link ref_48_link
- removed link ref_49_link
- removed link ref_4_link
- removed link ref_50_link
- removed link ref_51_link
- removed link ref_52_link
- removed link ref_53_link
- removed link ref_54_link
- removed link ref_55_link
- removed link ref_56_link
- removed link ref_57_link
- removed link ref_58_link
- removed link ref_59_link
- removed link ref_60_link
- removed link ref_61_link
- removed link ref_62_link
- removed link ref_63_link
- removed link ref_64_link
- removed link ref_65_link
- removed link ref_66_link
- removed link ref_67_link
- removed link ref_68_link
- removed link ref_69_link
- removed link ref_6_link
- removed link ref_70_link
- removed link ref_71_link
- removed link ref_72_link
- removed link ref_73_link
- removed link ref_74_link
- removed link ref_75_link
- removed link ref_76_link
- removed link ref_77_link
- removed link ref_78_link
- removed link ref_79_link
- removed link ref_7_link
- removed link ref_80_link
- removed link ref_81_link
- removed link ref_82_link
- removed link ref_83_link
- removed link ref_84_link
- removed link ref_85_link
- removed link ref_86_link
- removed link ref_87_link
- removed link ref_88_link
- removed link ref_89_link
- removed link ref_8_link
- removed link ref_90_link
- removed link ref_91_link
- removed link ref_92_link
- removed link ref_93_link
- removed link ref_94_link
- removed link ref_95_link
- removed link ref_96_link
- removed link ref_97_link
- removed link ref_98_link
- removed link ref_99_link
- added link body_link; visual box size=0.15 0.09 0.1
- added link l_wheel_link; visual cylinder length=0.028 radius=0.028
- added link r_wheel_link; visual cylinder length=0.028 radius=0.028
- link gyro_link: mass 0.023900 -> None; geometry visual box size=0.04 0.02 0.02
- link ultrasonic_link: mass 0.023900 -> None; geometry visual box size=0.02 0.055 0.02
Joints:
- removed joint m_wheel_joint
- removed joint ref_0_joint
- removed joint ref_100_joint
- removed joint ref_101_joint
- removed joint ref_102_joint
- removed joint ref_103_joint
- removed joint ref_104_joint
- removed joint ref_105_joint
- removed joint ref_10_joint
- removed joint ref_11_joint
- removed joint ref_12_joint
- removed joint ref_13_joint
- removed joint ref_14_joint
- removed joint ref_15_joint
- removed joint ref_16_joint
- removed joint ref_17_joint
- removed joint ref_18_joint
- removed joint ref_19_joint
- removed joint ref_1_joint
- removed joint ref_20_joint
- removed joint ref_21_joint
- removed joint ref_22_joint
- removed joint ref_23_joint
- removed joint ref_24_joint
- removed joint ref_25_joint
- removed joint ref_26_joint
- removed joint ref_27_joint
- removed joint ref_28_joint
- removed joint ref_29_joint
- removed joint ref_2_joint
- removed joint ref_30_joint
- removed joint ref_31_joint
- removed joint ref_32_joint
- removed joint ref_33_joint
- removed joint ref_34_joint
- removed joint ref_35_joint
- removed joint ref_36_joint
- removed joint ref_37_joint
- removed joint ref_38_joint
- removed joint ref_39_joint
- removed joint ref_3_joint
- removed joint ref_40_joint
- removed joint ref_41_joint
- removed joint ref_42_joint
- removed joint ref_43_joint
- removed joint ref_44_joint
- removed joint ref_45_joint
- removed joint ref_46_joint
- removed joint ref_47_joint
- removed joint ref_48_joint
- removed joint ref_49_joint
- removed joint ref_4_joint
- removed joint ref_50_joint
- removed joint ref_51_joint
- removed joint ref_52_joint
- removed joint ref_53_joint
- removed joint ref_54_joint
- removed joint ref_55_joint
- removed joint ref_56_joint
- removed joint ref_57_joint
- removed joint ref_58_joint
- removed joint ref_59_joint
- removed joint ref_5_joint
- removed joint ref_60_joint
- removed joint ref_61_joint
- removed joint ref_62_joint
- removed joint ref_63_joint
- removed joint ref_64_joint
- removed joint ref_65_joint
- removed joint ref_66_joint
- removed joint ref_67_joint
- removed joint ref_68_joint
- removed joint ref_69_joint
- removed joint ref_6_joint
- removed joint ref_70_joint
- removed joint ref_71_joint
- removed joint ref_72_joint
- removed joint ref_73_joint
- removed joint ref_74_joint
- removed joint ref_75_joint
- removed joint ref_76_joint
- removed joint ref_77_joint
- removed joint ref_78_joint
- removed joint ref_79_joint
- removed joint ref_7_joint
- removed joint ref_80_joint
- removed joint ref_81_joint
- removed joint ref_82_joint
- removed joint ref_83_joint
- removed joint ref_84_joint
- removed joint ref_85_joint
- removed joint ref_86_joint
- removed joint ref_87_joint
- removed joint ref_88_joint
- removed joint ref_89_joint
- removed joint ref_8_joint
- removed joint ref_90_joint
- removed joint ref_91_joint
- removed joint ref_92_joint
- removed joint ref_93_joint
- removed joint ref_94_joint
- removed joint ref_95_joint
- removed joint ref_96_joint
- removed joint ref_97_joint
- removed joint ref_98_joint
- removed joint ref_99_joint
- removed joint ref_9_joint
- added joint gyro_joint: type fixed, parent body_link, child gyro_link, origin xyz=-0.09 0 0.065 rpy=0 1.57079 0, axis 0 0 1
- added joint ultrasonic_joint: type fixed, parent body_link, child ultrasonic_link, origin xyz=0.06 0 -0.05 rpy=0 0 0, axis 0 0 1
- joint base_joint: child ref_0_link -> body_link; origin xyz=0.024 0 0.016 rpy=0 0 -1.57079632679 -> xyz=0 0 0.075 rpy=0 0 0
- joint l_wheel_joint: axis 1 0 0 -> 0 0 1; child ref_18_link_hub -> l_wheel_link; origin xyz=0 0 0 rpy=0 0 0 -> xyz=0.015 0.06 -0.05 rpy=-1.57079 0 0; parent ref_18_link -> body_link
- joint r_wheel_joint: axis 1 0 0 -> 0 0 -1; child ref_24_link_hub -> r_wheel_link; origin xyz=0 0 0 rpy=0 0 0 -> xyz=0.015 -0.06 -0.05 rpy=1.57079 0 0; parent ref_24_link -> body_link

Commit message: update rviz and urdf

File: ev3_robots/ev3_robot_gyro_car/robot.urdf (robot description, URDF)
Before this commit: robot ev3_robot_gyro_car, 6 links, 5 joints
Joints:
- joint gyro_joint: origin xyz=-0.09 0 0.065 rpy=0 1.57079 0 -> xyz=-0.09 0 0.065 rpy=0 0 0
